File: Hardware/KiCAD/bc_prace/bc_prace.kicad_sch (KiCad schematic)
At the start: 0 parts

Commit message: kicad
Other:
- sheet power renamed Power
- sheet Headphone Amp ports: added DAC_OUT_L, DAC_OUT_R; removed none
- sheet MCU ports: added LTC_KILL; removed none
- sheet Power ports: added CHG_DISABLE, LTC_KILL; removed CHG_ALLOW

Commit message: ioc, kicad
Other:
- added sheet User Interface (user_interface.kicad_sch)
- sheet DAC ports: added DAC_XSMT; removed none
- sheet MCU ports: added BTN_NEXT, BTN_PLAY, BTN_PREV, BTN_VOL_DOWN, BTN_VOL_UP, CHG_DISABLE, CHG_EN1, CHG_PGOOD, CHG_STATUS, DAC_XSMT, LTC_INT, OLED_CLK, OLED_CS, OLED_DC, OLED_MOSI, OLED_RST, VBUS_DET; removed none
- sheet Power ports: added LTC_INT, VBUS_DET; removed BAT_TEMP
