File: Hardware/KiCAD/bc_prace/dac.kicad_sch (KiCad schematic)
At the start: 15 parts, among them U5 PCM5102A

Commit message: ioc, kicad
Parts:
- added R35: 100K, Resistor_SMD:R_0805_2012Metric, symbol Device:R
Connections:
- net +3.3V: no longer U5.17 (XSMT)
- net GND: now also R35.1
- new net DAC_XSMT: R35.2, U5.17 (XSMT)
Other:
- note added: "C27 ověřit DC bias"
- note added: "C29 ověřit DC bias"
- note added: "firmware, pro soft-mute pro omezení prask/lup"
- moved on the sheet: C26, C27, C30, C31, C32, C33
