File: Hardware/KiCAD/bc_prace/headphone_amp.kicad_sch (KiCad schematic)
At the start: 12 parts, among them U6 TPA6111A2D

Commit message: kicad
Connections:
- net amp_shutdown renamed AMP_SHDW
Changed lines of the file:
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@@
 		(color 0 0 0 0)
 	)
-	(junction
-		(at 199.39 95.25)
-		(diameter 0)
-		(color 0 0 0 0)
-	)
 	(wire
 		(pts
@@
 	(wire
 		(pts
-			(xy 66.04 85.09) (xy 68.58 85.09)
-		)
-		(stroke
-			(width 0)
-			(type default)
-		)
-	)
-	(wire
-		(pts
 			(xy 227.33 76.2) (xy 227.33 54.61)
 		)
@@
 	(wire
 		(pts
-			(xy 199.39 95.25) (xy 200.66 95.25)
-		)
-		(stroke
-			(width 0)
-			(type default)
-		)
-	)
-	(wire
-		(pts
-			(xy 187.96 95.25) (xy 199.39 95.25)
+			(xy 187.96 95.25) (xy 200.66 95.25)
+		)
+		(stroke
+			(width 0)
+			(type default)
+		)
+	)
+	(wire
+		(pts
+			(xy 63.5 85.09) (xy 68.58 85.09)
 		)
 		(stroke
@@
 	(wire
 		(pts
-			(xy 199.39 97.79) (xy 199.39 95.25)
-		)
-		(stroke
-			(width 0)
-			(type default)
-		)
-	)
-	(wire
-		(pts
 			(xy 227.33 91.44) (xy 218.44 91.44)
-		)
-		(stroke
-			(width 0)
-			(type default)
-		)
-	)
-	(wire
-		(pts
-			(xy 200.66 97.79) (xy 199.39 97.79)
 		)
 		(stroke
@@
 		)
 	)
-	(global_label "DAC_OUT_R"
-		(shape input)
-		(at 247.65 91.44 0)
-		(fields_autoplaced yes)
-		(effects
-			(font
-				(size 1.27 1.27)
-			)
-			(justify left)
-		)
-		(property "Intersheetrefs" "${INTERSHEET_REFS}"
-			(at 261.0976 91.44 0)
-			(hide yes)
-			(show_name no)
-			(do_not_autoplace no)
-			(effects
-				(font
-					(size 1.27 1.27)
-				)
-				(justify left)
-			)
-		)
-	)
-	(global_label "amp_shutdown"
-		(shape input)
-		(at 200.66 95.25 0)
-		(fields_autoplaced yes)
-		(effects
-			(font
-				(size 1.27 1.27)
-			)
-			(justify left)
-		)
-		(property "Intersheetrefs" "${INTERSHEET_REFS}"
-			(at 217.4334 95.25 0)
-			(hide yes)
-			(show_name no)
-			(do_not_autoplace no)
-			(effects
-				(font
-					(size 1.27 1.27)
-				)
-				(justify left)
-			)
-		)
-	)
 	(global_label "HEADPHONE_OUT_R"
 		(shape input)
@@
 		)
 	)
-	(global_label "DAC_OUT_L"
+	(hierarchical_label "DAC_OUT_L"
 		(shape input)
-		(at 66.04 85.09 180)
-		(fields_autoplaced yes)
+		(at 63.5 85.09 180)
 		(effects
 			(font
@@
 			(justify right)
 		)
-		(property "Intersheetrefs" "${INTERSHEET_REFS}"
-			(at 52.8343 85.09 0)
-			(hide yes)
-			(show_name no)
-			(do_not_autoplace no)
-			(effects
-				(font
-					(size 1.27 1.27)
-				)
-				(justify right)
-			)
+	)
+	(hierarchical_label "DAC_OUT_R"
+		(shape input)
+		(at 247.65 91.44 0)
+		(effects
+			(font
+				(size 1.27 1.27)
+			)
+			(justify left)
 		)
 	)
 	(hierarchical_label "AMP_SHDW"
 		(shape input)
-		(at 200.66 97.79 0)
+		(at 200.66 95.25 0)
 		(effects
 			(font

Commit message: ioc, kicad
Parts:
- removed C35, C36: 470u, Capacitor_SMD:C_0805_2012Metric, symbol Device:C
- added C17, C18: 470u, Capacitor_SMD:CP_Elec_6.3x7.7, symbol Device:C_Polarized
- added D1: TPD2E1B06DRLR, Package_TO_SOT_SMD:SOT-563, symbol MP3_TI_ESD:TPD2E1B06DRLR
- added J3: SJ-3523-SMT-TR, Connector_Audio:Jack_3.5mm_CUI_SJ-3523-SMT_Horizontal, symbol Connector_Audio:AudioJack3
- R24, R25, R26, R27: value 10K -> 20K
- U6: footprint D8 -> Package_SO:SOIC-8_3.9x4.9mm_P1.27mm
Connections:
- net GND: now also D1.1 (IOA1), D1.4 (IOB2), J3.S
- net at R25.2, U6.1 (VO1): now also C18.1
- net at R27.1, U6.7 (VO2): now also C17.1
- new net: C17.2, D1.5 (IOA2), J3.R
- new net: C18.2, D1.2 (IOB1), J3.T
Other:
- note added: "0 V on high 3,3 OFF"
- note added: "potřeba obousměrné ESD ochrany, kmitá i pod 0V"
- note removed: "zpetnovazebni na 20 aby byl gain -0,5"
- moved on the sheet: C34, C37, C38, C39, C40, R24, R25, R26, R27, U6
