File: Hardware/KiCAD/bc_prace/power.kicad_sch (KiCad schematic)
At the start: 34 parts, among them J1 USB_C_Receptacle_USB2.0_16P, J2 BATTERY_RCY, J3 Conn_01x02, Q1 2N7002, U2 USBLC6-2SC6, U3 BQ24074RGT, U4 TPS63070RNMR

Commit message: kicad, cubemx, text
Parts:
- L1, U4: footprint Package_DFN_QFN:Texas_VQFN-HR-15_3x2.5mm_P0.5mm_Merged_7_8_AND_12_13 -> (none)
- R14: renamed from 5.1k; value R -> 5.1k
- R15: renamed from 5.1k; value R -> 5.1K
Connections:
- net VBUS: no longer names the net of C1.2, C4.2, J1.A4 (VBUS), J1.A9 (VBUS), J1.B4 (VBUS), J1.B9 (VBUS), U2.5 (VBUS), U3.13 (IN)
- net d_min: no longer names the net of J1.A7 (D-), J1.B7 (D-), U2.1 (I/O1)
- net d_plus: no longer names the net of J1.A6 (D+), J1.B6 (D+), U2.3 (I/O2)
Other:
- moved on the sheet: J1, R1, R14, R15, R8, R9

Commit message: kicad
Parts:
- removed J3: Conn_01x02, Package_DFN_QFN:VQFN-16-1EP_3x3mm_P0.5mm_EP1.6x1.6mm, symbol Connector_Generic:Conn_01x02
- removed Q1: 2N7002, Package_TO_SOT_SMD:SOT-23, symbol Transistor_FET:2N7002
- removed R4: 100K, Resistor_SMD:R_0805_2012Metric, symbol Device:R
- added C14: 100n, Capacitor_SMD:C_0805_2012Metric, symbol Device:C
- added C15: 1u, Capacitor_SMD:C_0805_2012Metric, symbol Device:C
- added C16: 330n, Capacitor_SMD:C_0805_2012Metric, symbol Device:C
- added R11, R29: 10K, Resistor_SMD:R_0805_2012Metric, symbol Device:R
- added R28, R30: 100K, Resistor_SMD:R_0805_2012Metric, symbol Device:R
- added SW1: POWER, Package_TO_SOT_SMD:TSOT-23-8, symbol Switch:SW_Push
- added U10: LTC2954ITS8-1, Package_TO_SOT_SMD:TSOT-23-8, symbol MP3_Power_Controllers:LTC2954ITS8-1
- added U9: TPD2E2U06DRL, Package_TO_SOT_SMD:SOT-553, symbol Power_Protection:TPD2E2U06DRL
- R3: value 47K -> 68K
Connections:
- net +3.3V: now also R29.1, R30.1
- net GND: now also R3.1, C14.1, C15.2, C16.2, R11.1, SW1.1, U10.4 (GND), U9.4
- net sys_power: now also C14.2, R28.2, U10.1 (VIN); no longer R3.1
- net at J1.A5 (CC1), R14.1: now also U9.3
- net at R10.1, U4.1 (PS/SYNC): no longer U4.14 (EN)
- net at J1.B5 (CC2), R15.2: now also U9.5
- net CHG_DISABLE: now reaches R3.2, U3.4 (~{CE})
- net BAT_TEMP: no longer names the net of U3.1 (TS)
- net BAT_TEMP: now also R11.2
- new net: SW1.2, U10.2 (PB)
- new net: C16.1, U10.3 (ONT)
- new net: C15.1, U10.7 (PDT)
- new net LTC_INT: R29.2, U10.5 (INT)
- new net LTC_KILL: R30.2, U10.8 (KILL)
- new net PWR_EN: R28.1, U10.6 (EN), U4.14 (EN)
- no-connect marks 5 -> 7
Other:
- note added: "default 32 ms ONT jinak 6,4s pro 1uF kondenzátor ke GND"
- note removed: "chg_allowed = 0V --> mosfet off, CE v log 1, nabíjení zakázáno chf_allowed = 3,3V --> mosfet ON, CE v log 0 nabijeni povoleno"
- moved on the sheet: C2, C3, C4, J2, R14, R15, R2, R5, R6, R7, R8, R9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

Commit message: ioc, kicad
Parts:
- added R33: 33K, Resistor_SMD:R_0805_2012Metric, symbol Device:R
- added R34: 82K, Resistor_SMD:R_0805_2012Metric, symbol Device:R
Connections:
- net GND: now also R34.2
- net at C1.2, C4.2, J1.A4 (VBUS)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: now also R33.1
- net BAT+ renamed bat_p
- new net VBUS_DET: R33.2, R34.1
Other:
- note added: "bat_m"
- moved on the sheet: C2, C3, C4, J2, R11, R2, R3, R5, R6, R7, R8, R9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
