File: Hardware/KiCAD/bc_prace/sd_card.kicad_sch (KiCad schematic)
At the start: 12 parts, among them J5 Micro_SD_Card_Det2, U7 USBLC6-4SC6, U8 USBLC6-4SC6

Commit message: ioc, kicad
Parts:
- C13: footprint Capacitor_SMD:C_0805_2012Metric -> Capacitor_SMD:C_1206_3216Metric
- J5: value Micro_SD_Card_Det2 -> DM3AT-SF-PEJM5; footprint Package_DFN_QFN:OnSemi_UDFN-16-1EP_1.35x3.3mm_P0.4mm_EP0.4x2.8mm -> Connector_Card:microSD_HC_Hirose_DM3AT-SF-PEJM5; symbol Connector:Micro_SD_Card_Det2 -> mp3_player:Micro_SD_Hirose_DM3AT
Connections:
- net GND: now also J5.11 (SHIELD); no longer J5.SH (SHIELD)
Other:
- note added: "C20 a C41 pouzdro 0805"
- note added: "C20 blízko pinu SD karty"
- note added: "bez karty log 1, na GND"
- note added: "c13 pouzdro 1206"
- note added: "karta IN - log 0,"
Changed lines of the file:
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@@
 	(generator_version "10.0")
 	(paper "A4")
+	(text "karta IN - log 0,"
+		(exclude_from_sim no)
+		(at 213.36 120.65 0)
+		(effects
+			(font
+				(size 1.27 1.27)
+			)
+		)
+	)
+	(text "C20 a C41 pouzdro 0805"
+		(exclude_from_sim no)
+		(at 162.56 27.178 0)
+		(effects
+			(font
+				(size 1.27 1.27)
+			)
+		)
+	)
+	(text "C20 blízko pinu SD karty"
+		(exclude_from_sim no)
+		(at 142.494 62.23 0)
+		(effects
+			(font
+				(size 1.27 1.27)
+			)
+		)
+	)
+	(text "c13 pouzdro 1206"
+		(exclude_from_sim no)
+		(at 158.242 24.13 0)
+		(effects
+			(font
+				(size 1.27 1.27)
+			)
+		)
+	)
+	(text "bez karty log 1, na GND"
+		(exclude_from_sim no)
+		(at 214.122 123.19 0)
+		(effects
+			(font
+				(size 1.27 1.27)
+			)
+		)
+	)
 	(junction
 		(at 107.95 57.15)
@@
 	)
 	(symbol
-		(lib_id "Connector:Micro_SD_Card_Det2")
+		(lib_id "mp3_player:Micro_SD_Hirose_DM3AT")
 		(at 240.03 88.9 0)
 		(unit 1)
@@
 			)
 		)
-		(property "Value" "Micro_SD_Card_Det2"
+		(property "Value" "DM3AT-SF-PEJM5"
 			(at 240.665 69.85 0)
 			(show_name no)
@@
 			)
 		)
-		(property "Footprint" "Package_DFN_QFN:OnSemi_UDFN-16-1EP_1.35x3.3mm_P0.4mm_EP0.4x2.8mm"
+		(property "Footprint" "Connector_Card:microSD_HC_Hirose_DM3AT-SF-PEJM5"
 			(at 292.1 71.12 0)
 			(hide yes)
@@
 		(pin "4"
 		)
-		(pin "SH"
+		(pin "11"
 		)
 		(pin "2"
@@
 			)
 		)
-		(property "Footprint" "Capacitor_SMD:C_0805_2012Metric"
+		(property "Footprint" "Capacitor_SMD:C_1206_3216Metric"
 			(at 129.54 46.6852 0)
 			(hide yes)
